File: proteusOBD2Ahonda.kicad_pcb (KiCad board)
At the start: 2 copper layers, 155 x 229.5 mm, 22 parts, among them J1 TE_179686-6_104pin_Connector, J2 Conn_01x08, J3 Conn_01x06, M1 Module-wbo-0.2, M2 Module-can-0.1, P1 Pad, Q1 Q_NIGBT_GCE

Commit message: Upd pinout
Parts:
- moved J2 122.8 mm to (259.1, 185.5)
- moved F1 122.8 mm to (242.8, 176.4)
- moved F2 122.8 mm to (229.9, 193.7)
- moved F3 122.8 mm to (234.5, 176.4)
- moved J3 122.8 mm to (228.1, 177.0)
- moved M1 122.8 mm to (226.5, 173.9)
- moved R1 122.8 mm to (285.7, 159.3)
- moved R2 122.8 mm to (235.8, 179.0)
- moved M2 122.8 mm to (247.6, 197.0)
- moved P1 122.8 mm to (232.3, 179.9)
- moved Q1 122.8 mm to (275.2, 164.5)
- moved BRD1 2.55 mm to (200.0, 84.1)

Commit message: Upd sch, pcb
Parts:
- removed F2, F3: Fuse-Pad-Pad, hellen-one-common:PAD-1206-PAD
- removed Q1: Q_NIGBT_GCE, Package_TO_SOT_SMD:TO-263-2
- added D1: SS34, Diode_SMD:D_SMA, F.Cu at (159.9, 80.2)
- added D2: SS34, Diode_SMD:D_SMA, F.Cu at (198.9, 80.4)
- added D3: SS34, Diode_SMD:D_SMA, F.Cu at (188.5, 217.8)
- added D4: SS34, Diode_SMD:D_SMA, F.Cu at (188.5, 212.8)
- added D5: SS34, Diode_SMD:D_SMA, F.Cu at (188.5, 202.8)
- added D6: SS34, Diode_SMD:D_SMA, F.Cu at (188.5, 207.8)
- added G2: PROTO_AREA, hellen-one-common:PROTO_AREA, F.Cu at (123.5, 239.7)
- added G3: PROTO_AREA, hellen-one-common:PROTO_AREA, F.Cu at (123.5, 252.4)
- added G4: PROTO_AREA, hellen-one-common:PROTO_AREA, F.Cu at (131.1, 239.7)
- added G5: PROTO_AREA, hellen-one-common:PROTO_AREA, F.Cu at (131.1, 252.4)
- added G6: PROTO_AREA, hellen-one-common:PROTO_AREA, F.Cu at (138.7, 227.0)
- added G7: PROTO_AREA, hellen-one-common:PROTO_AREA, F.Cu at (138.7, 252.4)
- added G8: PROTO_AREA, hellen-one-common:PROTO_AREA, F.Cu at (138.7, 239.7)
- added M2: Module-wbo-0.3, hellen-one-wbo-0.3:wbo, F.Cu at (82.6, 216.5)
- added P1: Pad, hellen-one-common:PAD-TH, F.Cu at (119.0, 79.3)
- added P10: Pad, hellen-one-common:PAD-TH, F.Cu at (116.0, 79.3)
- added P11: Pad, hellen-one-common:PAD-TH, F.Cu at (113.0, 79.3)
- added P12: Pad, hellen-one-common:PAD-TH, F.Cu at (107.0, 79.3)
- added P13: Pad, hellen-one-common:PAD-TH, F.Cu at (104.0, 79.3)
- added P14: Pad, hellen-one-common:PAD-TH, F.Cu at (92.0, 79.3)
- added P15: Pad, hellen-one-common:PAD-TH, F.Cu at (77.0, 79.3)
- added P16: Pad, hellen-one-common:PAD-TH, F.Cu at (71.0, 79.3)
- added P17: Pad, hellen-one-common:PAD-TH, F.Cu at (83.0, 79.3)
- added P18: Pad, hellen-one-common:PAD-TH, F.Cu at (80.0, 79.3)
- added P19: Pad, hellen-one-common:PAD-TH, F.Cu at (74.0, 79.3)
- added P2: Pad, hellen-one-common:PAD-TH, F.Cu at (98.0, 79.3)
- added P20: Pad, hellen-one-common:PAD-TH, F.Cu at (68.0, 79.3)
- added P22: Pad, hellen-one-common:PAD-TH, F.Cu at (179.0, 81.3)
- added P23: Pad, hellen-one-common:PAD-TH, F.Cu at (171.5, 81.3)
- added P24: Pad, hellen-one-common:PAD-TH, F.Cu at (194.0, 81.3)
- added P25: Pad, hellen-one-common:PAD-TH, F.Cu at (191.0, 81.3)
- added P26: Pad, hellen-one-common:PAD-TH, F.Cu at (188.0, 81.3)
- added P27: Pad, hellen-one-common:PAD-TH, F.Cu at (150.3, 80.8)
- added P28: Pad, hellen-one-common:PAD-TH, F.Cu at (182.0, 81.3)
- added P29: Pad, hellen-one-common:PAD-TH, F.Cu at (168.5, 81.3)
- added P3: Pad, hellen-one-common:PAD-TH, F.Cu at (95.0, 79.3)
- added P30: Pad, hellen-one-common:PAD-TH, F.Cu at (165.5, 81.3)
- added P31: Pad, hellen-one-common:PAD-TH, F.Cu at (194.0, 217.8)
- added P32: Pad, hellen-one-common:PAD-TH, F.Cu at (194.0, 212.8)
- added P33: Pad, hellen-one-common:PAD-TH, F.Cu at (194.0, 202.8)
- added P34: Pad, hellen-one-common:PAD-TH, F.Cu at (194.0, 207.8)
- added P35: Pad, hellen-one-common:PAD-TH, F.Cu at (201.5, 150.3)
- added P36: Pad, hellen-one-common:PAD-TH, F.Cu at (201.5, 147.3)
- added P37: Pad, hellen-one-common:PAD-TH, F.Cu at (201.5, 141.3)
- added P38: Pad, hellen-one-common:PAD-TH, F.Cu at (196.0, 105.8)
- added P39: Pad, hellen-one-common:PAD-TH, F.Cu at (196.0, 102.3)
- added P4: Pad, hellen-one-common:PAD-TH, F.Cu at (86.0, 79.3)
- added P40: Pad, hellen-one-common:PAD-TH, F.Cu at (196.0, 109.3)
- added P41: Pad, hellen-one-common:PAD-TH, F.Cu at (201.5, 109.8)
- added P42: Pad, hellen-one-common:PAD-TH, F.Cu at (201.5, 112.8)
- added P43: Pad, hellen-one-common:PAD-TH, F.Cu at (201.5, 118.3)
- added P44: Pad, hellen-one-common:PAD-TH, F.Cu at (201.5, 121.3)
- added P45: Pad, hellen-one-common:PAD-TH, F.Cu at (201.5, 126.3)
- added P46: Pad, hellen-one-common:PAD-TH, F.Cu at (201.5, 130.3)
- added P47: Pad, hellen-one-common:PAD-TH, F.Cu at (201.5, 133.3)
- added P48: Pad, hellen-one-common:PAD-TH, F.Cu at (201.5, 138.3)
- added P49: Pad, hellen-one-common:PAD-TH, F.Cu at (201.5, 144.3)
- added P5: Pad, hellen-one-common:PAD-TH, F.Cu at (122.0, 79.3)
- added P50: Pad, hellen-one-common:PAD-TH, F.Cu at (124.5, 169.8)
- added P51: Pad, hellen-one-common:PAD-TH, F.Cu at (127.5, 169.8)
- added P52: Pad, hellen-one-common:PAD-TH, F.Cu at (143.5, 169.8)
- added P53: Pad, hellen-one-common:PAD-TH, F.Cu at (134.5, 168.3)
- added P54: Pad, hellen-one-common:PAD-TH, F.Cu at (146.5, 169.8)
- added P55: Pad, hellen-one-common:PAD-TH, F.Cu at (149.5, 169.8)
- added P56: Pad, hellen-one-common:PAD-TH, F.Cu at (140.5, 169.8)
- added P57: Pad, hellen-one-common:PAD-TH, F.Cu at (137.5, 169.8)
- added P58: Pad, hellen-one-common:PAD-TH, F.Cu at (63.0, 118.3)
- added P59: Pad, hellen-one-common:PAD-TH, F.Cu at (63.0, 115.3)
- added P6: Pad, hellen-one-common:PAD-TH, F.Cu at (110.0, 79.3)
- added P60: Pad, hellen-one-common:PAD-TH, F.Cu at (63.0, 124.3)
- added P61: Pad, hellen-one-common:PAD-TH, F.Cu at (63.0, 121.3)
- added P62: Pad, hellen-one-common:PAD-TH, F.Cu at (63.0, 127.3)
- added P63: Pad, hellen-one-common:PAD-TH, F.Cu at (63.0, 130.3)
- added P64: Pad, hellen-one-common:PAD-TH, F.Cu at (63.0, 133.3)
- added P65: Pad, hellen-one-common:PAD-TH, F.Cu at (63.0, 146.8)
- added P7: Pad, hellen-one-common:PAD-TH, F.Cu at (101.0, 79.3)
- added P8: Pad, hellen-one-common:PAD-TH, F.Cu at (89.0, 79.3)
- added P9: Pad, hellen-one-common:PAD-TH, F.Cu at (125.0, 79.3)
- added R3: 4.7k, hellen-one-common:R0603, F.Cu at (112.0, 83.3)
- added R4: 4.7k, hellen-one-common:R0603, F.Cu at (103.3, 83.3)
- added R5: 4.7k, hellen-one-common:R0603, F.Cu at (99.0, 83.3)
- added R6: 4.7k, hellen-one-common:R0603, F.Cu at (116.5, 83.3)
- added R7: 4.7k, hellen-one-common:R0603, F.Cu at (107.5, 83.3)
- added R8: 4.7k, hellen-one-common:R0603, F.Cu at (94.5, 83.3)
- added R9: 1k, hellen-one-common:R1206, F.Cu at (174.2, 80.9)
- J2: value Conn_01x08 -> XH-10AW; footprint hellen-one-common:XH-8A -> Connector_JST:JST_XH_S10B-XH-A_1x10_P2.50mm_Horizontal
- M1: value Module-wbo-0.2 -> Module-vr-discrete-0.1; footprint hellen-one-wbo-0.2:wbo -> hellen-one-vr-discrete-0.1:vr-discrete
- R1, R2: value Res -> Jumper-Pad-Pad; footprint hellen-one-common:R0603 -> hellen-one-common:PAD-0805-PAD
- moved J2 200.5 mm to (74.2, 263.0)
- moved R1 176.6 mm to (127.5, 80.8), turned to -90 degrees
- moved J4 159.2 mm to (78.0, 230.0), turned to 180 degrees
- moved M3 150.4 mm to (97.6, 207.6), turned to 180 degrees
- moved F1 131.2 mm to (153.3, 80.4), turned to -90 degrees
- moved R2 114.8 mm to (176.5, 80.8), turned to -90 degrees
- moved P21 109.4 mm to (185.0, 81.3)
- moved M1 56.8 mm to (177.7, 203.0), turned to 90 degrees
- renumbered J3 to J4, M2 to M3, P1 to P21
Connections:
- F1 pad 1: unconnected-(F1-Pad1) -> Net-(F1-Pad1)
- F1 pad 2: /12V_MR -> /12V
- J1 pad A1: (no net) -> /OUT_INJ4
- J1 pad A10: (no net) -> GND
- J1 pad A11: (no net) -> Net-(F1-Pad1)
- J1 pad A12: (no net) -> /OUT_IDLE
- J1 pad A13: (no net) -> Net-(J1-PadA13)
- J1 pad A14: (no net) -> Net-(J1-PadA14)
- J1 pad A15: (no net) -> Net-(J1-PadA15)
- J1 pad A16: (no net) -> /OUT_FUEL_PUMP
- J1 pad A17: (no net) -> /OUT_CONDITIONER_CLUTCH
- J1 pad A18: (no net) -> /OUT_CHECK_ENGINE
- J1 pad A19: (no net) -> Net-(J1-PadA19)
- J1 pad A2: (no net) -> /OUT_INJ3
- J1 pad A20: (no net) -> /OUT_IGN_CONTROL
- J1 pad A22: (no net) -> GND
- J1 pad A23: (no net) -> GND
- J1 pad A24: (no net) -> Net-(J1-PadA24)
- J1 pad A27: (no net) -> /OUT_FAN
- J1 pad A28: (no net) -> Net-(J1-PadA28)
- J1 pad A29: (no net) -> Net-(J1-PadA29)
- J1 pad A3: (no net) -> /OUT_INJ2
- J1 pad A30: (no net) -> Net-(J1-PadA30)
- J1 pad A4: (no net) -> /OUT_INJ1
- J1 pad A5: (no net) -> Net-(J1-PadA5)
- J1 pad A6: (no net) -> Net-(J1-PadA6)
- J1 pad A7: (no net) -> Net-(J1-PadA7)
- J1 pad A8: (no net) -> /OUT_VTEC
- J1 pad A9: (no net) -> GND
- J1 pad C1: (no net) -> /IN_CRANK_FLUCT
- J1 pad C10: (no net) -> Net-(J1-PadC10)
- J1 pad C11: (no net) -> Net-(J1-PadC11)
- J1 pad C12: (no net) -> /IN_CRANK-
- J1 pad C13: (no net) -> Net-(J1-PadC13)
- J1 pad C14: (no net) -> /IN_CYP-
- J1 pad C15: (no net) -> /IN_OIL_PRESSURE
- J1 pad C16: (no net) -> /IN_STEERING
- J1 pad C17: (no net) -> Net-(J1-PadC17)
- J1 pad C18: (no net) -> /IN_VSS
- J1 pad C19: (no net) -> Net-(J1-PadC19)
- J1 pad C2: (no net) -> /IN_CRANK+
- J1 pad C21: (no net) -> Net-(J1-PadC21)
- J1 pad C23: (no net) -> Net-(J1-PadC23)
- J1 pad C24: (no net) -> Net-(J1-PadC24)
- J1 pad C25: (no net) -> Net-(J1-PadC25)
- J1 pad C27: (no net) -> Net-(J1-PadC27)
- J1 pad C28: (no net) -> Net-(J1-PadC28)
- J1 pad C29: (no net) -> /IN_AT_PARK/CLUTCH
- J1 pad C3: (no net) -> Net-(J1-PadC3)
- J1 pad C30: (no net) -> Net-(J1-PadC30)
- J1 pad C4: (no net) -> /IN_CYP+
- J1 pad C5: (no net) -> /IN_AC_REQUEST
- J1 pad C6: (no net) -> /IN_STARTER_SW
- J1 pad C7: (no net) -> /IN_SERVICE_CHECK
- J1 pad C8: (no net) -> Net-(J1-PadC8)
- J1 pad C9: (no net) -> Net-(J1-PadC9)
- J1 pad D1: (no net) -> /IN_TPS
- J1 pad D10: (no net) -> +5V
- J1 pad D11: (no net) -> GND
- J1 pad D12: (no net) -> GND
- J1 pad D13: (no net) -> Net-(J1-PadD13)
- J1 pad D14: (no net) -> Net-(J1-PadD14)
- J1 pad D15: (no net) -> Net-(J1-PadD15)
- J1 pad D16: (no net) -> Net-(J1-PadD16)
- J1 pad D2: (no net) -> /IN_CLT
- J1 pad D3: (no net) -> /IN_MAP
- J1 pad D4: (no net) -> +5V
- J1 pad D5: (no net) -> /IN_BRAKE
- J1 pad D6: (no net) -> /IN_KNOCK
- J1 pad D7: (no net) -> Net-(J1-PadD7)
- J1 pad D8: (no net) -> /IN_IAT
- J1 pad D9: (no net) -> Net-(J1-PadD9)
- J2 pad 1: GND -> /12V
- J2 pad 2: GND -> /12V
- J2 pad 3: /WBO_H- -> /WBO_Vs
- J2 pad 4: /WBO_H- -> /WBO_Vs/Ip
- J2 pad 5: /WBO_R_Trim -> /WBO_Ip
- J2 pad 6: /WBO_Ip -> /WBO_R_Trim
- J2 pad 7: /WBO_Vs/Ip -> /WBO_H-
- J2 pad 8: /WBO_Vs -> /WBO_H-
- J4 pad 1: Net-(J3-Pad1) -> Net-(J4-Pad1)
- J4 pad 2: Net-(J3-Pad2) -> Net-(J4-Pad2)
- J4 pad 4: Net-(J3-Pad4) -> Net-(J4-Pad4)
- J4 pad 5: Net-(J3-Pad5) -> Net-(J4-Pad5)
- M1 pad E1: /WBO_Vs -> /VR_THRESH
- M1 pad E2: /WBO_Vs/Ip -> (no net)
- M1 pad E3: /WBO_Ip -> Net-(M1-PadE3)
- M1 pad E4: /WBO_R_Trim -> +5V
- M1 pad W1: /5V_SENSOR_2 -> /IN_CYP-
- M1 pad W2: Net-(M1-PadW2) -> /IN_CYP+
- M3 pad S1: (no net) -> Net-(M3-PadS1)
- M3 pad S2: (no net) -> Net-(M3-PadS2)
- M3 pad V1: /5V_SENSOR_2 -> +5V
- M3 pad V2: Net-(M1-PadW2) -> Net-(M2-PadW2)
- M3 pad V5: Net-(M1-PadW4) -> Net-(M2-PadW4)
- M3 pad V6: Net-(M1-PadW3) -> Net-(M2-PadW3)
- P21 pad 1: (no net) -> Net-(J1-PadA5)
- R1 pad 1: Net-(Q1-Pad1) -> Net-(J1-PadC11)
- R1 pad 2: /GATE_IGN1 -> +5V
- R2 pad 1: /GATE_IGN1 -> Net-(J1-PadA19)
- R2 pad 2: /OUT_IGN1 -> /OUT_ALTERN_CONTROL
Other:
- board text added: "+12V"
- board text added: "C"
- board text added: "D"
- board text added: "G"
- board text added: "GND"
- board text added: "H-"
- board text added: "Ip"
- board text added: "R_Trim"
- board text added: "SWD:R"
- board text added: "V"
- board text added: "Vs"
- board text added: "Vs/Ip"
- board text added: "WBO1"

Commit message: Upd pcb
Parts:
- added J5: Conn_01x01, TestPoint:TestPoint_Pad_D2.0mm, B.Cu at (119.0, 175.0)
- moved M1 70.5 mm to (110.2, 182.5), turned to -90 degrees
- moved D3 18.2 mm to (185.5, 199.8)
- moved D4 18.2 mm to (185.5, 194.8)
- moved D5 18.2 mm to (185.5, 184.8)
- moved D6 18.2 mm to (185.5, 189.8)
- moved P31 18.2 mm to (191.0, 199.8)
- moved P32 18.2 mm to (191.0, 194.8)
- moved P33 18.2 mm to (191.0, 184.8)
- moved P34 18.2 mm to (191.0, 189.8)
- moved P35 6.30 mm to (195.2, 150.4)
- moved P36 6.30 mm to (195.2, 147.4)
- moved P37 6.30 mm to (195.2, 141.4)
- moved P49 6.30 mm to (195.2, 144.4)
- moved R3 4.50 mm to (107.5, 83.3), turned to 180 degrees
- moved R7 4.50 mm to (112.0, 83.3)
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Routing:
- net /12V: track 0.00 -> 451.4 mm, vias 0 -> 8
- net +5V: track 0.00 -> 288.9 mm, vias 0 -> 5
- net /VR_THRESH: track 0.00 -> 158.1 mm, vias 0 -> 5
- net +12V_PROT: track 0.00 -> 143.1 mm, vias 0 -> 2
- net /IN_BRAKE: track 0.00 -> 129.2 mm, vias 0 -> 1
- net /IN_CYP-: track 0.00 -> 114.1 mm
- net /IN_AT_PARK/CLUTCH: track 0.00 -> 110.6 mm, vias 0 -> 1
- net /IN_CYP+: track 0.00 -> 109.3 mm
- net /IN_STARTER_SW: track 0.00 -> 101.7 mm, vias 0 -> 1
- net /IN_VSS: track 0.00 -> 100.3 mm, vias 0 -> 1
- net Net-(BRD1-PadA20(16)): track 0.00 -> 97.8 mm, vias 0 -> 1
- net Net-(BRD1-PadA9(4)): track 0.00 -> 96.8 mm, vias 0 -> 1
- net /OUT_VTEC: track 0.00 -> 96.1 mm, vias 0 -> 1
- net Net-(BRD1-PadA10(3)): track 0.00 -> 94.0 mm, vias 0 -> 1
- net /IN_CRANK-: track 0.00 -> 90.4 mm
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- added copper zone on B.Cu, net GND
- added copper zone on F.Cu, net GND
Other:
- board text added: "12V"
- board text added: "5V"

Commit message: UPD pcb
Parts:
- added G***: LOGO, LOGO, F.Cu at (168.5, 252.0)
- moved G1 38.5 mm to (146.0, 267.0)
Routing:
- net Net-(BRD1-PadB4(5)): track 19.9 -> 19.2 mm
Other:
- board text added: "Proteus Honda OBD2A adapter rev. a"
- board text added: "https://rusefi.com/s/proteus-honda-obd2a"

Commit message: Fab preview
Parts:
- added R10: Jumper-Pad-Pad, hellen-one-common:PAD-0805-PAD, F.Cu at (125.5, 81.0)
- added R11: Jumper-Pad-Pad, hellen-one-common:PAD-0805-PAD, F.Cu at (120.5, 81.0)
- added R12: Jumper-Pad-Pad, hellen-one-common:PAD-0805-PAD, F.Cu at (115.5, 81.0)
- added R13: Jumper-Pad-Pad, hellen-one-common:PAD-0805-PAD, F.Cu at (108.0, 81.0)
- added R14: Jumper-Pad-Pad, hellen-one-common:PAD-0805-PAD, F.Cu at (105.5, 81.0)
- added R15: Jumper-Pad-Pad, hellen-one-common:PAD-0805-PAD, F.Cu at (100.5, 81.0)
- added R16: Jumper-Pad-Pad, hellen-one-common:PAD-0805-PAD, F.Cu at (123.0, 81.0)
- added R17: Jumper-Pad-Pad, hellen-one-common:PAD-0805-PAD, F.Cu at (118.0, 81.0)
- added R18: Jumper-Pad-Pad, hellen-one-common:PAD-0805-PAD, F.Cu at (113.0, 81.0)
- added R19: Jumper-Pad-Pad, hellen-one-common:PAD-0805-PAD, F.Cu at (110.5, 81.0)
- added R20: Jumper-Pad-Pad, hellen-one-common:PAD-0805-PAD, F.Cu at (103.0, 81.0)
- added R21: Jumper-Pad-Pad, hellen-one-common:PAD-0805-PAD, F.Cu at (95.5, 81.0)
- added R22: Jumper-Pad-Pad, hellen-one-common:PAD-0805-PAD, F.Cu at (165.0, 81.0)
- added R23: Jumper-Pad-Pad, hellen-one-common:PAD-0805-PAD, F.Cu at (197.0, 81.0)
- added R24: Jumper-Pad-Pad, hellen-one-common:PAD-0805-PAD, F.Cu at (185.0, 81.0)
- added R25: Jumper-Pad-Pad, hellen-one-common:PAD-0805-PAD, F.Cu at (182.5, 81.0)
- added R26: Jumper-Pad-Pad, hellen-one-common:PAD-0805-PAD, F.Cu at (180.0, 81.0)
- added R27: Jumper-Pad-Pad, hellen-one-common:PAD-0805-PAD, F.Cu at (172.0, 81.0)
- added R28: Jumper-Pad-Pad, hellen-one-common:PAD-0805-PAD, F.Cu at (187.0, 81.0)
- added R29: Jumper-Pad-Pad, hellen-one-common:PAD-0805-PAD, F.Cu at (111.0, 205.5)
- moved P11 14.5 mm to (116.0, 93.5)
- moved P12 10.7 mm to (109.5, 90.0)
- moved P13 10.7 mm to (103.5, 90.0)
- moved P6 10.7 mm to (106.5, 90.0)
- moved P7 10.7 mm to (100.5, 90.0)
- moved P10 9.70 mm to (116.0, 89.0)
- moved P30 8.26 mm to (168.5, 89.0)
- moved P21 8.10 mm to (187.5, 89.0)
- moved P22 7.72 mm to (178.5, 89.0)
- moved P23 7.72 mm to (172.0, 89.0)
- moved P28 7.70 mm to (182.0, 89.0)
- moved P9 7.15 mm to (127.5, 86.0)
- moved P1 6.72 mm to (118.5, 86.0)
- moved P5 6.72 mm to (121.5, 86.0)
- moved P4 5.12 mm to (90.0, 82.5)
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Connections:
- BRD1 pad C10(3): (no net) -> unconnected-(BRD1-PadC10(3))
- BRD1 pad C22(14): (no net) -> unconnected-(BRD1-PadC22(14))
- BRD1 pad C33(26): (no net) -> unconnected-(BRD1-PadC33(26))
- D1 pad 1: /12V -> /OUT_VTEC
- D1 pad 2: /OUT_VTEC -> GND
- J1 pad A12: /OUT_IDLE -> Net-(J1-PadA12)
- J1 pad A16: /OUT_FUEL_PUMP -> Net-(J1-PadA16)
- J1 pad A17: /OUT_CONDITIONER_CLUTCH -> Net-(J1-PadA17)
- J1 pad A18: /OUT_CHECK_ENGINE -> Net-(J1-PadA18)
- J1 pad A20: /OUT_IGN_CONTROL -> Net-(J1-PadA20)
- J1 pad A21: (no net) -> unconnected-(J1-PadA21)
- J1 pad A25: (no net) -> unconnected-(J1-PadA25)
- J1 pad A26: (no net) -> unconnected-(J1-PadA26)
- J1 pad A27: /OUT_FAN -> Net-(J1-PadA27)
- J1 pad A31: (no net) -> unconnected-(J1-PadA31)
- J1 pad A32: (no net) -> unconnected-(J1-PadA32)
- J1 pad A8: /OUT_VTEC -> Net-(J1-PadA8)
- J1 pad B1: (no net) -> unconnected-(J1-PadB1)
- J1 pad B10: (no net) -> unconnected-(J1-PadB10)
- J1 pad B11: (no net) -> unconnected-(J1-PadB11)
- J1 pad B12: (no net) -> unconnected-(J1-PadB12)
- J1 pad B13: (no net) -> unconnected-(J1-PadB13)
- J1 pad B14: (no net) -> unconnected-(J1-PadB14)
- J1 pad B15: (no net) -> unconnected-(J1-PadB15)
- J1 pad B16: (no net) -> unconnected-(J1-PadB16)
- J1 pad B17: (no net) -> unconnected-(J1-PadB17)
- J1 pad B18: (no net) -> unconnected-(J1-PadB18)
- J1 pad B19: (no net) -> unconnected-(J1-PadB19)
- J1 pad B2: (no net) -> unconnected-(J1-PadB2)
- J1 pad B20: (no net) -> unconnected-(J1-PadB20)
- J1 pad B21: (no net) -> unconnected-(J1-PadB21)
- J1 pad B22: (no net) -> unconnected-(J1-PadB22)
- J1 pad B23: (no net) -> unconnected-(J1-PadB23)
- J1 pad B24: (no net) -> unconnected-(J1-PadB24)
- J1 pad B25: (no net) -> unconnected-(J1-PadB25)
- J1 pad B3: (no net) -> unconnected-(J1-PadB3)
- J1 pad B4: (no net) -> unconnected-(J1-PadB4)
- J1 pad B5: (no net) -> unconnected-(J1-PadB5)
- J1 pad B6: (no net) -> unconnected-(J1-PadB6)
- J1 pad B7: (no net) -> unconnected-(J1-PadB7)
- J1 pad B8: (no net) -> unconnected-(J1-PadB8)
- J1 pad B9: (no net) -> unconnected-(J1-PadB9)
- J1 pad C1: /IN_CRANK_FLUCT -> Net-(J1-PadC1)
- J1 pad C12: /IN_CRANK- -> Net-(J1-PadC12)
- J1 pad C14: /IN_CYP- -> Net-(J1-PadC14)
- J1 pad C15: /IN_OIL_PRESSURE -> Net-(J1-PadC15)
- J1 pad C16: /IN_STEERING -> Net-(J1-PadC16)
- J1 pad C18: /IN_VSS -> Net-(J1-PadC18)
- J1 pad C2: /IN_CRANK+ -> Net-(J1-PadC2)
- J1 pad C20: (no net) -> unconnected-(J1-PadC20)
- J1 pad C22: (no net) -> unconnected-(J1-PadC22)
- J1 pad C26: (no net) -> unconnected-(J1-PadC26)
- J1 pad C29: /IN_AT_PARK/CLUTCH -> Net-(J1-PadC29)
- J1 pad C31: (no net) -> unconnected-(J1-PadC31)
- J1 pad C4: /IN_CYP+ -> Net-(J1-PadC4)
- J1 pad C5: /IN_AC_REQUEST -> Net-(J1-PadC5)
- J1 pad C6: /IN_STARTER_SW -> Net-(J1-PadC6)
- J1 pad C7: /IN_SERVICE_CHECK -> Net-(J1-PadC7)
- J4 pad 6: (no net) -> unconnected-(J4-Pad6)
- M1 pad E1: /VR_THRESH -> Net-(M1-PadE1)
- M1 pad E2: (no net) -> unconnected-(M1-PadE2)
- M2 pad J2: (no net) -> unconnected-(M2-PadJ2)
- M2 pad J_GND2: (no net) -> unconnected-(M2-PadJ_GND2)
- M2 pad J_VCC1: (no net) -> unconnected-(M2-PadJ_VCC1)
- M2 pad J_VCC2: (no net) -> unconnected-(M2-PadJ_VCC2)
Routing:
- net Net-(J1-PadC25): track 13.4 -> 30.9 mm
- net /OUT_FAN: track 42.4 -> 25.1 mm
- net /IN_AT_PARK/CLUTCH: track 110.6 -> 94.3 mm
- net Net-(J1-PadC29): track 0.00 -> 13.5 mm
- net Net-(J1-PadA27): track 0.00 -> 13.5 mm
- net Net-(J1-PadC28): track 13.8 -> 27.1 mm
- net /IN_CRANK-: track 90.1 -> 76.9 mm
- net /IN_VSS: track 100.3 -> 87.0 mm
- net Net-(J1-PadC19): track 8.64 -> 21.6 mm
- net /IN_STEERING: track 66.8 -> 53.9 mm
- net Net-(J1-PadC24): track 13.3 -> 26.2 mm
- net /IN_OIL_PRESSURE: track 63.7 -> 51.0 mm
- net /OUT_CHECK_ENGINE: track 57.7 -> 45.2 mm
- net /OUT_CONDITIONER_CLUTCH: track 59.7 -> 47.3 mm
- net /OUT_FUEL_PUMP: track 43.4 -> 31.2 mm
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