File: proteusOBD2Ahonda.kicad_sch (KiCad schematic)
At the start: 16 parts, among them J2 XH-8A, J3 Conn_01x06, M1 Module-wbo-0.2, M2 Module-can-0.1, P1 Pad, Q1 ISL9V3040S3S

Commit message: Outline
Parts:
- added G1: RUSEFI_LOGO, kicad6-libraries:rusefi_logo, symbol rusefi_logo:RUSEFI_LOGO
- added H1, H2, H3, H4, H5, H6, H7, H8: MountingHole, MountingHole:MountingHole_4.3mm_M4, symbol Mechanical:MountingHole
- F2: LCSC (none) -> C182446; MyComment DNP -> (none)
- F3: value 10A -> Fuse-Pad-Pad; footprint hellen-one-common:36911600000 -> hellen-one-common:PAD-1206-PAD; LCSC C354908 -> C182446
- J2: value XH-8A -> Conn_01x08; LCSC C10385 -> (none)
- Q1: value ISL9V3040S3S -> Q_NIGBT_GCE; LCSC C898702 -> (none)
- R1: value 22 -> Res; LCSC C23345 -> (none)
- R2: value DNP -> Res; footprint Resistor_SMD:R_2512_6332Metric -> hellen-one-common:R0603
- gave numbers to parts that had none: 2

Commit message: Upd pinout
Parts:
- removed M1: Module-wbo-0.2, hellen-one-wbo-0.2:wbo, symbol hellen-one-wbo-0.2:Module-wbo-0.2
- added D? (x2): SS34, Diode_SMD:D_SMA, symbol Device:D_Schottky
- added F?: Fuse-Pad-Pad, hellen-one-common:PAD-1206-PAD, symbol hellen-one-common:Fuse-Pad-Pad
- added M?: Module-wbo-0.3, hellen-one-wbo-0.3:wbo, symbol hellen-one-wbo-0.3:Module-wbo-0.3
- added M?: Module-vr-discrete-0.1, hellen-one-vr-discrete-0.1:vr-discrete, symbol hellen-one-vr-discrete-0.1:Module-vr-discrete-0.1
- added P? (x20): Pad, hellen-one-common:PAD-TH, symbol hellen-one-common:Pad
- added R? (x6): 4.7k, hellen-one-common:R0603, symbol hellen-one-common:Res
- added R?: 1k, hellen-one-common:R1206, symbol hellen-one-common:Res
- added R? (x2): Jumper-Pad-Pad, hellen-one-common:PAD-0805-PAD, symbol hellen-one-common:Jumper-Pad-Pad
- renumbered BRD1 to BRD?, F3 to F?, F2 to F?, F1 to F?, G1 to G?, H5 to H?, H7 to H?, H4 to H?, H3 to H?, H1 to H?, H6 to H?, H8 to H?, H2 to H?, J2 to J?, J1 to J?, J3 to J?, M2 to M?, P1 to P?, Q1 to Q?, R1 to R?, R2 to R?
Connections:
- net 5V_SENSOR_2: now also M?.W1 (V5_IN)
- net GND: now also J?.A10, J?.A22, J?.A23, J?.A9, J?.D11, J?.D12, M?.E6 (LSU_H-), M?.G (GND)
- net IN_KNOCK: now also BRD?.C34 (KNOCK1), J?.D6
- net WBO_H-: now also M?.E5 (LSU_H+)
- net WBO_Ip: now also M?.E3 (LSU_Ip)
- net WBO_R_Trim: now also M?.E4 (LSU_Rtrim)
- net WBO_Vs: now also M?.E1 (LSU_Un)
- net WBO_Vs/Ip: now also M?.E2 (LSU_Vm)
- net OUT_FAN: now reaches BRD?.A12 (LS15(FAN))
- net OUT_FAN: now also J?.A27
- net OUT_INJ2: now reaches BRD?.A15 (LS2(INJ2))
- net OUT_INJ2: now also J?.A3
- net OUT_INJ4: now reaches BRD?.A16 (LS4(INJ4))
- net OUT_INJ4: now also J?.A1
- net OUT_VTEC: now reaches BRD?.A2 (HS1)
- net OUT_VTEC: now also J?.A8, D?.2 (A)
- net OUT_FUEL_PUMP: now reaches BRD?.A23 (LS16(FUEL))
- net OUT_FUEL_PUMP: now also J?.A16
- net OUT_INJ1: now reaches BRD?.A3 (LS1(INJ1))
- net OUT_INJ1: now also J?.A4
- net OUT_INJ3: now reaches BRD?.A4 (LS3(INJ3))
- net OUT_INJ3: now also J?.A2
- net 12V_IGN: now reaches BRD?.B18 (12V_IGN)
- net 12V_IGN: now also F?.2, R?.2, R?.2, R?.2, R?.2, R?.2, R?.2
- net IN_MAP: now reaches BRD?.C13 (AV1(MAP))
- net IN_MAP: now also J?.D3
- net IN_CLT: now reaches BRD?.C20 (AT3(CLT))
- net IN_CLT: now also J?.D2
- net IN_TPS: now reaches BRD?.C24 (AV2(TPS))
- net IN_TPS: now also J?.D1
- net IN_IAT: now reaches BRD?.C30 (AT2(IAT))
- net IN_IAT: now also J?.D8
- net at J?.A11: now also F?.1
- net OUT_IDLE: now reaches J?.A12
- net OUT_IDLE: now also D?.2 (A)
- net at J?.A15: now also P?.1 (Pin_1)
- net OUT_CONDITIONER_CLUTCH: now reaches J?.A17
- net OUT_CHECK_ENGINE: now reaches J?.A18
- net at J?.A19: now also R?.1
- net OUT_IGN_CONTROL: now reaches J?.A20
- net OUT_IGN_CONTROL: now also R?.1
- net at J?.A24: now also P?.1 (Pin_1)
- net at J?.A28: now also P?.1 (Pin_1)
- net at J?.A29: now also P?.1 (Pin_1)
- net at J?.A30: now also P?.1 (Pin_1)
- net at J?.A5: now also P?.1 (Pin_1)
- net at J?.A6: now also P?.1 (Pin_1)
- net at J?.A7: now also P?.1 (Pin_1)
- net at M?.V2 (CAN_VIO): now also M?.W2 (CAN_VIO)
- net at M?.V6 (CAN_RX): now also M?.W3 (CAN_RX)
- net at M?.V5 (CAN_TX): now also M?.W4 (CAN_TX)
- net at J?.5 (Pin_5): now also M?.W5 (nReset)
- net at J?.4 (Pin_4): now also M?.W6 (SWDIO)
- net at J?.2 (Pin_2): now also M?.W7 (SWCLK)
- net at J?.1 (Pin_1): now also M?.W8 (V33_OUT)
- net IN_CRANK_FLUCT: now reaches J?.C1
- net at J?.C10: now also P?.1 (Pin_1)
- net at J?.C11: now also R?.1
- net IN_CRANK-: now reaches J?.C12
- net at J?.C13: now also P?.1 (Pin_1)
- net IN_CYP-: now reaches J?.C14
- net IN_OIL_PRESSURE: now reaches J?.C15
- net IN_OIL_PRESSURE: now also R?.1
- net IN_STEERING: now reaches J?.C16
- net IN_STEERING: now also R?.1
- net at J?.C17: now also P?.1 (Pin_1)
- net IN_VSS: now reaches J?.C18
- net at J?.C19: now also P?.1 (Pin_1)
- net IN_CRANK+: now reaches J?.C2
- net at J?.C21: now also P?.1 (Pin_1)
- net at J?.C27: now also P?.1 (Pin_1)
- net at J?.C28: now also P?.1 (Pin_1)
- net AT_PARK/CLUTCH: now reaches J?.C29
- net AT_PARK/CLUTCH: now also R?.1
- net at J?.C3: now also P?.1 (Pin_1)
- net at J?.C30: now also P?.1 (Pin_1)
- net IN_CYP+: now reaches J?.C4
- net IN_AC_REQUEST: now reaches J?.C5
- net IN_AC_REQUEST: now also R?.1
- net IN_STARTER_SW: now reaches J?.C6
- net IN_STARTER_SW: now also R?.1
- net IN_SERVICE_CHECK: now reaches J?.C7
- net IN_SERVICE_CHECK: now also R?.1
- net at J?.C8: now also P?.1 (Pin_1)
- net at J?.C9: now also P?.1 (Pin_1)
- net +5V: now reaches J?.D10
- net +5V: now also J?.D4, R?.2
- net at J?.D15: now also P?.1 (Pin_1)
- net at J?.D16: now also P?.1 (Pin_1)
- net IN_BRAKE: now reaches J?.D5
- net IN_EGR_LIFT: now reaches J?.D9
- new net: M?.J1 (SEL1), M?.J_GND1 (PULL_DOWN1)
- new net OUT_ALTERN_CONTROL: R?.2
- no-connect marks 5 -> 41
Other:
- note added: "12V BATT"
- note added: "12V_IGN"
- note added: "AT Check"
- note added: "Alternator field"
- note added: "Baro output???"
- note added: "IDLE???"
- moved on the sheet: BRD?, P?

Commit message: Upd sch, pcb
Parts:
- removed F? (x3): Fuse-Pad-Pad, hellen-one-common:PAD-1206-PAD, symbol hellen-one-common:Fuse-Pad-Pad
- removed J?: Conn_01x08, hellen-one-common:XH-8A, symbol Connector_Generic:Conn_01x08
- removed M?: Module-vr-discrete-0.1, hellen-one-vr-discrete-0.1:vr-discrete, symbol hellen-one-vr-discrete-0.1:Module-vr-discrete-0.1
- removed Q?: Q_NIGBT_GCE, Package_TO_SOT_SMD:TO-263-2, symbol Device:Q_NIGBT_GCE
- removed R? (x2): Res, hellen-one-common:R0603, symbol hellen-one-common:Res
- added D3, D4, D5, D6: SS34, Diode_SMD:D_SMA, symbol Device:D_Schottky
- added G2, G3, G4, G5, G6, G7, G8: PROTO_AREA, hellen-one-common:PROTO_AREA, symbol hellen-one-common:PROTO_AREA
- added J2: XH-10AW, Connector_JST:JST_XH_S10B-XH-A_1x10_P2.50mm_Horizontal, symbol Connector_Generic:Conn_01x10
- added J3: XH-10A, Connector_JST:JST_XH_B10B-XH-A_1x10_P2.50mm_Vertical, symbol Connector_Generic:Conn_01x10
- added M1: Module-vr-discrete-0.1, hellen-one-vr-discrete-0.1:vr-discrete, symbol hellen-one-vr-discrete-0.1:Module-vr-discrete-0.1
- added P10, P11, P15, P16, P17, P18, P24, P25, P31, P32, P33, P34, P35, P36, P37, P38, P39, P40, P41, P42, P43, P44, P45, P46, P47, P48, P49, P50, P51, P52, P53, P54, P55, P56, P57, P58, P59, P60, P61, P62, P63, P64, P65, P9: Pad, hellen-one-common:PAD-TH, symbol hellen-one-common:Pad
- gave numbers to parts that had none: 47
Connections:
- net 5V_SENSOR_2 is gone; now on net +5V: M2.W1 (V5_IN), M3.V1 (V5)
- net +5V: now also BRD1.C21(15) (5V_1), BRD1.C32(27) (5V_1), BRD1.C9(4) (5V_1), G6.10, G6.6, G6.7, G6.8, G6.9, M1.E4 (V5_IN)
- net GND: now also BRD1.A17(19) (GND), BRD1.A18(18) (GND), BRD1.A24(35) (GND), BRD1.B14(10) (GND), BRD1.B19(20) (GND), BRD1.B20(19) (GND), BRD1.C1(12) (GND_SENS), BRD1.C2(11) (GND_SENS), BRD1.C23(13) (GND_SENS), BRD1.C29(30) (GND_SENS), BRD1.C3(10) (GND_SENS), BRD1.C4(9) (GND_SENS), BRD1.C5(8) (GND_SENS), BRD1.C6(7) (GND_SENS), BRD1.C7(6) (GND_SENS), BRD1.C8(5) (GND_SENS), G6.1, G6.2, G6.3, G6.4, G6.5, J2.10 (Pin_10), J2.9 (Pin_9), J3.10 (Pin_10), J3.9 (Pin_9), M1.G (GND)
- net IN_AC_REQUEST: now also BRD1.C26(33) (AV6)
- net IN_BRAKE: now also BRD1.B10(14) (D1)
- net IN_CLT: now also BRD1.C20(16) (AT3(CLT)); no longer BRD1.C20 (AT3(CLT))
- net IN_CRANK+: now also BRD1.B5(4) (VR1+)
- net IN_CRANK-: now also BRD1.B13(11) (VR1-)
- net IN_CRANK_FLUCT: now also BRD1.B2(7) (D3)
- net IN_CYP+: now also M1.W2 (VR+)
- net IN_CYP-: now also M1.W1 (VR-)
- net IN_IAT: now also BRD1.C30(29) (AT2(IAT)); no longer BRD1.C30 (AT2(IAT))
- net IN_KNOCK: now also BRD1.C34(25) (KNOCK1); no longer BRD1.C34 (KNOCK1)
- net IN_MAP: now also BRD1.C13(23) (AV1(MAP)); no longer BRD1.C13 (AV1(MAP))
- net IN_OIL_PRESSURE: now also BRD1.C25(34) (AV4)
- net IN_SERVICE_CHECK: now also BRD1.C15(21) (AV5)
- net IN_STARTER_SW: now also BRD1.B3(6) (D4)
- net IN_STEERING: now also BRD1.C14(22) (AV3)
- net IN_TPS: now also BRD1.C24(35) (AV2(TPS)); no longer BRD1.C24 (AV2(TPS))
- net IN_VSS: now also BRD1.B1(8) (D2)
- net OUT_ALTERN_CONTROL: now also BRD1.A5(8) (LS5(INJ5))
- net OUT_CHECK_ENGINE: now also BRD1.A7(6) (LS7(INJ7))
- net OUT_CONDITIONER_CLUTCH: now also BRD1.A19(17) (LS8(INJ8))
- net OUT_FAN: now also BRD1.A12(1) (LS15(FAN)); no longer BRD1.A12 (LS15(FAN))
- net OUT_FUEL_PUMP: now also BRD1.A23(13) (LS16(FUEL)); no longer BRD1.A23 (LS16(FUEL))
- net OUT_IDLE: now also BRD1.A6(7) (LS6(INJ6))
- net OUT_IGN_CONTROL: now also BRD1.A8(5) (LS9(INJ9))
- net OUT_INJ1: now also BRD1.A3(10) (LS1(INJ1)); no longer BRD1.A3 (LS1(INJ1))
- net OUT_INJ2: now also BRD1.A15(21) (LS2(INJ2)); no longer BRD1.A15 (LS2(INJ2))
- net OUT_INJ3: now also BRD1.A4(9) (LS3(INJ3)); no longer BRD1.A4 (LS3(INJ3))
- net OUT_INJ4: now also BRD1.A16(20) (LS4(INJ4)); no longer BRD1.A16 (LS4(INJ4))
- net OUT_VTEC: now also BRD1.A2(11) (HS1); no longer BRD1.A2 (HS1)
- net WBO_H-: now also J2.7 (Pin_7), J2.8 (Pin_8), J3.7 (Pin_7), J3.8 (Pin_8)
- net WBO_Ip: now also J2.5 (Pin_5), J3.5 (Pin_5)
- net WBO_R_Trim: now also J2.6 (Pin_6), J3.6 (Pin_6)
- net WBO_Vs: now also J2.3 (Pin_3), J3.3 (Pin_3)
- net WBO_Vs/Ip: now also J2.4 (Pin_4), J3.4 (Pin_4)
- net at J1.A13: now also P24.1 (Pin_1)
- net at J1.A14: now also P25.1 (Pin_1)
- net 12V: now reaches D1.1 (K)
- net 12V: now also BRD1.B18(21) (12V_IGN), BRD1.B23(16) (12V_MR), D2.1 (K), F1.2, R3.2, R4.2, R5.2, R6.2, R7.2, R8.2, R9.2, D3.1 (K), D4.1 (K), D5.1 (K), D6.1 (K), J2.1 (Pin_1), J2.2 (Pin_2), J3.1 (Pin_1), J3.2 (Pin_2)
- net at J1.C23: now also P9.1 (Pin_1)
- net at J1.C24: now also P10.1 (Pin_1)
- net at J1.C25: now also P11.1 (Pin_1)
- net at J1.D13: now also P17.1 (Pin_1)
- net at J1.D14: now also P18.1 (Pin_1)
- net at J1.D7: now also P15.1 (Pin_1)
- removed net 12V_IGN: BRD1.B18 (12V_IGN), F1.2, R3.2, R4.2, R5.2, R6.2, R7.2, R8.2
- net AT_PARK/CLUTCH renamed IN_AT_PARK/CLUTCH
- net IN_AT_PARK/CLUTCH: now also BRD1.B9(15) (D5)
- net CAN_H: no longer names the net of M3.S2 (CANH)
- net CAN_H: now also BRD1.B17(22) (CAN+)
- net CAN_L: no longer names the net of M3.S1 (CANL)
- net CAN_L: now also BRD1.B16(23) (CAN-)
- net IN_EGR_LIFT: no longer names the net of J1.D9
- net IN_EGR_LIFT: now also P16.1 (Pin_1)
- new net: BRD1.C28(31) (AV10), P61.1 (Pin_1)
- new net: BRD1.A1(12) (HS2), P35.1 (Pin_1)
- new net: BRD1.A10(3) (LS13(MAIN)), D6.2 (A), P34.1 (Pin_1)
- new net: BRD1.A11(2) (LS14), P38.1 (Pin_1)
- new net: BRD1.A13(23) (HS3), P36.1 (Pin_1)
- new net: BRD1.A14(22) (HS4), P37.1 (Pin_1)
- new net: BRD1.A20(16) (LS10(INJ10)), D3.2 (A), P31.1 (Pin_1)
- new net: BRD1.A21(15) (LS12(INJ12)), D5.2 (A), P33.1 (Pin_1)
- new net: BRD1.A22(14) (IGN3), P41.1 (Pin_1)
- new net: BRD1.A25(34) (IGN12), P49.1 (Pin_1)
- new net: BRD1.A26(33) (IGN11), P48.1 (Pin_1)
- new net: BRD1.A27(32) (IGN10), P47.1 (Pin_1)
- new net: BRD1.A28(31) (IGN9), P46.1 (Pin_1)
- new net: BRD1.A29(30) (IGN8), P45.1 (Pin_1)
- new net: BRD1.A30(29) (IGN7), P44.1 (Pin_1)
- new net: BRD1.A31(28) (IGN6), P43.1 (Pin_1)
- new net: BRD1.A33(26) (IGN4), P42.1 (Pin_1)
- new net: BRD1.A34(25) (IGN2), P40.1 (Pin_1)
- new net: BRD1.A35(24) (IGN1), P39.1 (Pin_1)
- new net: BRD1.A9(4) (LS11(INJ11)), D4.2 (A), P32.1 (Pin_1)
- new net: BRD1.B11(13) (D6), M1.E3 (OUT)
- new net: BRD1.B12(12) (VR2-), P51.1 (Pin_1)
- new net: BRD1.B15(9) (ETB2+), P54.1 (Pin_1)
- new net: BRD1.B21(18) (CAN2-), P57.1 (Pin_1)
- new net: BRD1.B22(17) (CAN2+), P56.1 (Pin_1)
- new net: BRD1.B4(5) (VR2+), P50.1 (Pin_1)
- new net: BRD1.B6(3) (ETB1-), P53.1 (Pin_1)
- new net: BRD1.B7(2) (ETB1+), P52.1 (Pin_1)
- new net: BRD1.B8(1) (ETB2-), P55.1 (Pin_1)
- new net: BRD1.C16(20) (AV7), P58.1 (Pin_1)
- new net: BRD1.C17(19) (AV9), P60.1 (Pin_1)
- new net: BRD1.C18(18) (AV11), P62.1 (Pin_1)
- new net: BRD1.C19(17) (AT1), P63.1 (Pin_1)
- new net: BRD1.C27(32) (AV8), P59.1 (Pin_1)
- new net: BRD1.C31(28) (AT4), P64.1 (Pin_1)
- new net: BRD1.C35(24) (KNOCK2), P65.1 (Pin_1)
- new net: G5.1, G5.11, G5.6
- new net: G5.10, G5.15, G5.5
- new net: G5.12, G5.2, G5.7
- new net: G5.13, G5.3, G5.8
- new net: G5.14, G5.4, G5.9
- new net: G7.1, G7.11, G7.6
- new net: G7.10, G7.15, G7.5
- new net: G7.12, G7.2, G7.7
- new net: G7.13, G7.3, G7.8
- new net: G7.14, G7.4, G7.9
- new net: G3.1, G3.11, G3.6
- new net: G3.10, G3.15, G3.5
- new net: G3.12, G3.2, G3.7
- new net: G3.13, G3.3, G3.8
- new net: G3.14, G3.4, G3.9
- new net: G4.1, G4.11, G4.6
- new net: G4.10, G4.15, G4.5
- new net: G4.12, G4.2, G4.7
- new net: G4.13, G4.3, G4.8
- new net: G4.14, G4.4, G4.9
- new net: G8.1, G8.11, G8.6
- new net: G8.10, G8.15, G8.5
- new net: G8.12, G8.2, G8.7
- new net: G8.13, G8.3, G8.8
- new net: G8.14, G8.4, G8.9
- new net: G2.1, G2.11, G2.6
- new net: G2.10, G2.15, G2.5
- new net: G2.12, G2.2, G2.7
- new net: G2.13, G2.3, G2.8
- new net: G2.14, G2.4, G2.9
- new net +12V_PROT: BRD1.C11(2) (12V_PROT), BRD1.C12(1) (12V_PROT), G6.11, G6.12, G6.13, G6.14, G6.15
- new net VR_THRESH: BRD1.A32(27) (IGN5), M1.E1 (Thresh_IN)
- no-connect marks 41 -> 42
Other:
- note removed: "Example"
- note removed: "IDLE???"
- moved on the sheet: D1, D2, F1, J1A, J1B, J1C, J1D, J4, M2, M3, P1, P12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

Commit message: Upd pcb
Parts:
- added J5: Conn_01x01, TestPoint:TestPoint_Pad_D2.0mm, symbol Connector_Generic:Conn_01x01
Connections:
- net GND: now also J5.1 (Pin_1)
Changed lines of the file:
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@@
+    (pin "1")
+  )
+  (symbol (lib_id "power:GND") (at 44.45 400.05 0) (unit 1)
+    (in_bom yes) (on_board yes)
+    (property "Reference" "#PWR05" (id 0) (at 44.45 406.4 0)
+      (effects (font (size 1.27 1.27)) hide)
+    )
+    (property "Value" "GND" (id 1) (at 44.5008 403.9934 0))
+    (property "Footprint" "" (id 2) (at 44.45 400.05 0)
+      (effects (font (size 1.27 1.27)) hide)
+    )
+    (property "Datasheet" "" (id 3) (at 44.45 400.05 0)
+      (effects (font (size 1.27 1.27)) hide)
+    )
     (pin "1")
   )
@@
     )
     (property "Datasheet" "~" (id 3) (at 45.72 133.35 0)
+      (effects (font (size 1.27 1.27)) hide)
+    )
+    (pin "1")
+  )
+  (symbol (lib_id "Connector_Generic:Conn_01x01") (at 49.53 400.05 0) (unit 1)
+    (in_bom yes) (on_board yes)
+    (property "Reference" "J5" (id 0) (at 51.562 400.1516 0)
+      (effects (font (size 1.27 1.27)) (justify left))
+    )
+    (property "Value" "Conn_01x01" (id 1) (at 51.562 401.2946 0)
+      (effects (font (size 1.27 1.27)) (justify left) hide)
+    )
+    (property "Footprint" "TestPoint:TestPoint_Pad_D2.0mm" (id 2) (at 49.53 400.05 0)
+      (effects (font (size 1.27 1.27)) hide)
+    )
+    (property "Datasheet" "~" (id 3) (at 49.53 400.05 0)
       (effects (font (size 1.27 1.27)) hide)
     )
@@
       (reference "#PWR04") (unit 1) (value "+12V_PROT") (footprint "")
     )
+    (path "/5ba5bd90-704f-4bb1-8228-d568c909d17f"
+      (reference "#PWR05") (unit 1) (value "GND") (footprint "")
+    )
     (path "/35fdad3f-2c21-454f-befd-3065d541bff8"
       (reference "#PWR0101") (unit 1) (value "GND") (footprint "")
@@
       (reference "J4") (unit 1) (value "Conn_01x06") (footprint "Connector_PinHeader_2.54mm:PinHeader_1x06_P2.54mm_Vertical")
     )
+    (path "/6504a4bb-e6b7-488a-895d-2786ec342012"
+      (reference "J5") (unit 1) (value "Conn_01x01") (footprint "TestPoint:TestPoint_Pad_D2.0mm")
+    )
     (path "/761d8935-faf5-4823-98ff-382292025f5c"

Commit message: UPD pcb
Connections:
- net 12V: no longer D1.1 (K)
- net GND: now also D1.2 (A)
- net OUT_VTEC: now also D1.1 (K); no longer D1.2 (A)
Other:
- note added: "https://rusefi.com/s/proteus-honda-obd2a"
- moved on the sheet: D1, J5

Commit message: Fab preview
Parts:
- added R10, R11, R12, R13, R14, R15, R16, R17, R18, R19, R20, R21, R22, R23, R24, R25, R26, R27, R28, R29: Jumper-Pad-Pad, hellen-one-common:PAD-0805-PAD, symbol hellen-one-common:Jumper-Pad-Pad
Connections:
- net IN_AC_REQUEST: now also R13.2; no longer J1.C5
- net IN_AT_PARK/CLUTCH: now also R21.2; no longer J1.C29
- net IN_CRANK+: now also R11.2; no longer J1.C2
- net IN_CRANK-: now also R16.2; no longer J1.C12
- net IN_CRANK_FLUCT: now also R10.2; no longer J1.C1
- net IN_CYP+: now also R12.2; no longer J1.C4
- net IN_CYP-: now also R17.2; no longer J1.C14
- net IN_OIL_PRESSURE: now also R18.2; no longer J1.C15
- net IN_SERVICE_CHECK: now also R15.2; no longer J1.C7
- net IN_STARTER_SW: now also R14.2; no longer J1.C6
- net IN_STEERING: now also R19.2; no longer J1.C16
- net IN_VSS: now also R20.2; no longer J1.C18
- net OUT_CHECK_ENGINE: now also R26.2; no longer J1.A18
- net OUT_CONDITIONER_CLUTCH: now also R25.2; no longer J1.A17
- net OUT_FAN: now also R28.2; no longer J1.A27
- net OUT_FUEL_PUMP: now also R24.2; no longer J1.A16
- net OUT_IDLE: now also R23.2; no longer J1.A12
- net OUT_IGN_CONTROL: now also R27.2; no longer J1.A20
- net OUT_VTEC: now also R22.2; no longer J1.A8
- net VR_THRESH: now also R29.2; no longer M1.E1 (Thresh_IN)
- new net: J1.A27, R28.1
- new net: J1.A12, R23.1
- new net: J1.A16, R24.1
- new net: J1.A17, R25.1
- new net: J1.A18, R26.1
- new net: J1.A20, R27.1
- new net: J1.A8, R22.1
- new net: J1.C12, R16.1
- new net: J1.C15, R18.1
- new net: M1.E1 (Thresh_IN), R29.1
- new net: J1.C29, R21.1
- new net: J1.C1, R10.1
- new net: J1.C14, R17.1
- new net: J1.C16, R19.1
- new net: J1.C18, R20.1
- new net: J1.C2, R11.1
- new net: J1.C4, R12.1
- new net: J1.C5, R13.1
- new net: J1.C6, R14.1
- new net: J1.C7, R15.1
- no-connect marks 42 -> 43
Other:
- moved on the sheet: R9
